File: PCB/pico/chord_pico.kicad_pcb (KiCad board)
At the start: 2 copper layers, 268.8 x 136.9 mm, 83 parts, among them SW1 SW_DIP_x01, SW2 SW_DIP_x01, U1 PiPico, U2 ADG706BRUZ, U6 LM4040DBZ-3, U7 TPS7A2042

Commit message: PCB progress 60%
Parts:
- removed JP2: Bypass, Jumper:SolderJumper-2_P1.3mm_Open_RoundedPad1.0x1.5mm
- added C21: 0.1uF, Capacitor_SMD:C_0603_1608Metric_Pad1.08x0.95mm_HandSolder, F.Cu at (184.2, 175.1)
- added C22: 0.1uF, Capacitor_SMD:C_0603_1608Metric_Pad1.08x0.95mm_HandSolder, F.Cu at (204.2, 175.1)
- added C23: 0.1uF, Capacitor_SMD:C_0603_1608Metric_Pad1.08x0.95mm_HandSolder, F.Cu at (224.2, 175.1)
- added C24: 0.1uF, Capacitor_SMD:C_0603_1608Metric_Pad1.08x0.95mm_HandSolder, F.Cu at (244.2, 175.1)
- added C25: 0.1uF, Capacitor_SMD:C_0603_1608Metric_Pad1.08x0.95mm_HandSolder, F.Cu at (264.2, 175.1)
- added C26: 0.1uF, Capacitor_SMD:C_0603_1608Metric_Pad1.08x0.95mm_HandSolder, F.Cu at (284.2, 175.1)
- added C27: 0.1uF, Capacitor_SMD:C_0603_1608Metric_Pad1.08x0.95mm_HandSolder, F.Cu at (304.2, 175.1)
- added C28: 0.1uF, Capacitor_SMD:C_0603_1608Metric_Pad1.08x0.95mm_HandSolder, F.Cu at (324.2, 175.1)
- added CC1: 0.1uF, Capacitor_SMD:C_0603_1608Metric_Pad1.08x0.95mm_HandSolder, B.Cu at (191.7, 187.2)
- added CC2: 0.1uF, Capacitor_SMD:C_0603_1608Metric_Pad1.08x0.95mm_HandSolder, B.Cu at (191.7, 190.5)
- C1, C10, C11, C12, C2, C3, C4, C5, C6, C7, C8, C9, H1, H10, H11, H12, H2, H3, H4, H5, H6, H7, H8, H9: moved to F.Cu
- moved C15 130.8 mm to (260.3, 105.3), turned to 180 degrees
- moved C16 130.8 mm to (280.3, 105.3), turned to 180 degrees
- moved C17 80.6 mm to (104.2, 175.1)
- moved C18 80.6 mm to (124.2, 175.1)
- moved C19 80.6 mm to (144.2, 175.1)
- moved C20 80.6 mm to (164.2, 175.1)
- moved C13 70.2 mm to (140.3, 105.3), turned to 180 degrees
- moved C14 70.2 mm to (160.3, 105.3), turned to 180 degrees
- moved C6 6.97 mm to (208.0, 205.5), turned to 0 degrees
- moved C10 6.88 mm to (287.5, 210.4), turned to 0 degrees
- moved C11 6.88 mm to (307.5, 215.4), turned to 0 degrees
- moved C9 6.88 mm to (267.8, 207.1), turned to 0 degrees
- moved C12 6.88 mm to (332.5, 224.3), turned to 0 degrees
- moved C2 6.88 mm to (128.5, 215.4), turned to 0 degrees
- moved C3 6.88 mm to (148.5, 210.4), turned to 0 degrees
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Connections:
- C10 pad 1: +5V -> Vref
- C11 pad 1: +5V -> Vref
- C12 pad 1: +5V -> Vref
- C13 pad 1: +5V -> Vref
- C14 pad 1: +5V -> Vref
- C15 pad 1: +5V -> Vref
- C16 pad 1: +5V -> Vref
- C20 pad 1: Vref -> +5V
- C8 pad 1: /V1 -> Vref
- C9 pad 1: /V2 -> Vref
- H1 pad 2: /K2 -> /K1
- H13 pad 3: Net-(H13-G) -> GND
- H14 pad 3: Net-(H13-G) -> GND
- H15 pad 3: Net-(H13-G) -> GND
- H16 pad 3: Net-(H13-G) -> GND
- H2 pad 2: /K3 -> /K2
- H3 pad 2: /K4 -> /K3
- H4 pad 2: /K6 -> /K4
- H5 pad 2: /K1 -> /K5
- H6 pad 2: /K5 -> /K6
- SW1 pad 2: Net-(SW1-Pad2) -> GND
- SW2 pad 2: Net-(SW1-Pad2) -> GND
- U1 pad 1: /AUX1 -> Net-(D1-In)
- U1 pad 17: Net-(D1-In) -> unconnected-(U1-GPIO13-Pad17)
- U1 pad 19: unconnected-(U1-GPIO14-Pad19) -> /AUX1
- U1 pad 2: /AUX2 -> unconnected-(U1-GPIO1-Pad2)
- U1 pad 20: unconnected-(U1-GPIO15-Pad20) -> /AUX2
- U2 pad 10: /K10 -> /K8
- U2 pad 11: /K9 -> /K7
- U2 pad 13: (no net) -> unconnected-(U2-NC-Pad13)
- U2 pad 19: /K1 -> /K6
- U2 pad 2: (no net) -> unconnected-(U2-NC-Pad2)
- U2 pad 20: /K2 -> /K5
- U2 pad 21: /K3 -> /K4
- U2 pad 22: /K4 -> /K3
- U2 pad 23: /K5 -> /K2
- U2 pad 24: /K6 -> /K1
- U2 pad 25: /K7 -> /F1
- U2 pad 26: /K8 -> /F2
- U2 pad 3: (no net) -> unconnected-(U2-NC-Pad3)
- U2 pad 4: unconnected-(U2-S16-Pad4) -> /F3
- U2 pad 5: /F3 -> /F4
- U2 pad 6: unconnected-(U2-S14-Pad6) -> /K12
- U2 pad 7: /F1 -> /K11
- U2 pad 8: /K12 -> /K10
- U2 pad 9: /K11 -> /K9
Routing:
- net Vref: track 0.00 -> 433.0 mm, vias 0 -> 2
- net Net-(D1-In): track 0.00 -> 139.2 mm, vias 0 -> 1
- net /F4: track 0.00 -> 139.1 mm
- net /F1: track 0.00 -> 138.3 mm
- net /F3: track 0.00 -> 130.3 mm
- net /F2: track 0.00 -> 128.9 mm
- net /K1: track 0.00 -> 127.2 mm, vias 0 -> 1
- net /K12: track 0.00 -> 122.0 mm, vias 0 -> 1
- net /AUX2: track 0.00 -> 116.9 mm, vias 0 -> 1
- net /AUX1: track 0.00 -> 108.5 mm, vias 0 -> 1
- net Net-(U1-VBUS): track 0.00 -> 105.8 mm, vias 0 -> 2
- net /K2: track 0.00 -> 98.3 mm, vias 0 -> 1
- net /K11: track 0.00 -> 93.0 mm, vias 0 -> 1
- net Net-(U1-USB1): track 0.00 -> 85.9 mm
- net Net-(U1-USB2): track 0.00 -> 85.3 mm
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
Commit message: PCB v1.0
Parts:
- added CC3: 0.1uF, Capacitor_SMD:C_0603_1608Metric_Pad1.08x0.95mm_HandSolder, B.Cu at (228.2, 193.8)
- R4: value 10K -> 5.1K
- moved U2 8.00 mm to (222.2, 198.1)
- moved C1 3.96 mm to (100.4, 221.8)
- moved C2 3.50 mm to (126.5, 212.5)
- moved C3 3.47 mm to (146.3, 207.8)
- moved C11 3.10 mm to (305.5, 213.0)
- moved C5 3.10 mm to (186.0, 203.1)
- moved C6 3.10 mm to (206.0, 203.1)
- moved C7 3.10 mm to (226.0, 203.1)
- moved C8 3.10 mm to (246.0, 203.1)
- moved C9 3.10 mm to (265.8, 204.7)
- moved C4 3.10 mm to (166.3, 204.7)
- moved C10 2.89 mm to (285.8, 208.1)
- moved C12 2.19 mm to (331.6, 222.3)
- moved C13 1.40 mm to (140.3, 103.9)
- moved C14 1.40 mm to (160.3, 103.9)
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Connections:
- U2 pad 14: Net-(U1-GPIO18) -> Net-(U1-GPIO17)
- U2 pad 15: Net-(U1-GPIO19) -> Net-(U1-GPIO18)
- U2 pad 16: Net-(U1-GPIO20) -> Net-(U1-GPIO19)
- U2 pad 17: Net-(U1-GPIO21) -> Net-(U1-GPIO20)
- U2 pad 18: Net-(U1-GPIO17) -> Net-(U1-GPIO21)
Routing:
- net +5V: track 55.5 -> 906.7 mm, vias 0 -> 1
- net Vref: track 433.0 -> 658.4 mm, vias 2 -> 4
- net Net-(U1-GPIO17): track 0.00 -> 32.6 mm
- net Net-(U1-GPIO18): track 0.00 -> 30.3 mm
- net Net-(U1-GPIO19): track 0.00 -> 27.2 mm
- net Net-(U1-GPIO20): track 0.00 -> 24.1 mm
- net Net-(U1-GPIO21): track 0.00 -> 21.7 mm
- net GND: track 4.14 -> 25.7 mm, vias 1 -> 144
- net /F2: track 128.9 -> 139.6 mm
- net /F1: track 138.3 -> 147.7 mm
- net /K9: track 49.3 -> 42.2 mm
- net /K8: track 28.6 -> 21.5 mm
- net /K11: track 93.0 -> 85.9 mm
- net /K1: track 127.2 -> 134.3 mm
- net Net-(U2-D): track 2.87 -> 9.85 mm
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- added copper zone on B.Cu, net GND
- added copper zone on F.Cu, net GND
Other:
- outline, holes or cut-outs redrawn
- board text added: "Chord Pico"
- board text added: "v1.0"

Commit message: PCB v1.11
Parts:
- removed C13, C14, C15, C16: 0.1uF, Capacitor_SMD:C_0603_1608Metric_Pad1.08x0.95mm_HandSolder
- removed H13, H14, H15, H16: SS49E_SOT23, Package_TO_SOT_THT:TO-92Flat
- added C29: 0.1uF, Capacitor_SMD:C_0603_1608Metric_Pad1.08x0.95mm_HandSolder, F.Cu at (127.2, 120.6)
- added C30: 0.1uF, Capacitor_SMD:C_0603_1608Metric_Pad1.08x0.95mm_HandSolder, F.Cu at (181.2, 120.6)
- added C31: 0.1uF, Capacitor_SMD:C_0603_1608Metric_Pad1.08x0.95mm_HandSolder, F.Cu at (247.2, 120.6)
- added C32: 0.1uF, Capacitor_SMD:C_0603_1608Metric_Pad1.08x0.95mm_HandSolder, F.Cu at (301.2, 120.6)
- added D35: WS2812B_Unified, chord_pico:WS2812B-2835, F.Cu at (124.7, 115.1)
- added D36: WS2812B_Unified, chord_pico:WS2812B-2835, F.Cu at (183.7, 115.1)
- added D37: WS2812B_Unified, chord_pico:WS2812B-2835, F.Cu at (244.7, 115.1)
- added D38: WS2812B_Unified, chord_pico:WS2812B-2835, F.Cu at (303.7, 115.1)
- added D39: WS2812B_Unified, chord_pico:WS2812B-2835, F.Cu at (119.2, 115.1)
- added D40: WS2812B_Unified, chord_pico:WS2812B-2835, F.Cu at (189.2, 115.1)
- added D41: WS2812B_Unified, chord_pico:WS2812B-2835, F.Cu at (239.2, 115.1)
- added D42: WS2812B_Unified, chord_pico:WS2812B-2835, F.Cu at (309.2, 115.1)
- added IR1: ITR1502, chord_pico:ITR1502, F.Cu at (134.2, 102.1)
- added IR10: ITR1502, chord_pico:ITR1502, F.Cu at (294.2, 102.1)
- added IR2: ITR1502, chord_pico:ITR1502, F.Cu at (144.2, 102.1)
- added IR3: ITR1502, chord_pico:ITR1502, F.Cu at (154.2, 102.1)
- added IR4: ITR1502, chord_pico:ITR1502, F.Cu at (164.2, 102.1)
- added IR5: ITR1502, chord_pico:ITR1502, F.Cu at (174.2, 102.1)
- added IR6: ITR1502, chord_pico:ITR1502, F.Cu at (254.2, 102.1)
- added IR7: ITR1502, chord_pico:ITR1502, F.Cu at (264.2, 102.1)
- added IR8: ITR1502, chord_pico:ITR1502, F.Cu at (274.2, 102.1)
- added IR9: ITR1502, chord_pico:ITR1502, F.Cu at (284.2, 102.1)
- added R10: 10K, Resistor_SMD:R_0603_1608Metric_Pad0.98x0.95mm_HandSolder, F.Cu at (154.0, 106.1)
- added R11: 200, Resistor_SMD:R_0603_1608Metric_Pad0.98x0.95mm_HandSolder, F.Cu at (168.7, 100.5)
- added R12: 10K, Resistor_SMD:R_0603_1608Metric_Pad0.98x0.95mm_HandSolder, F.Cu at (164.0, 106.1)
- added R13: 200, Resistor_SMD:R_0603_1608Metric_Pad0.98x0.95mm_HandSolder, F.Cu at (178.7, 100.4)
- added R14: 10K, Resistor_SMD:R_0603_1608Metric_Pad0.98x0.95mm_HandSolder, F.Cu at (174.0, 106.1)
- added R15: 200, Resistor_SMD:R_0603_1608Metric_Pad0.98x0.95mm_HandSolder, F.Cu at (258.7, 100.5)
- added R16: 10K, Resistor_SMD:R_0603_1608Metric_Pad0.98x0.95mm_HandSolder, F.Cu at (254.0, 106.1)
- added R17: 200, Resistor_SMD:R_0603_1608Metric_Pad0.98x0.95mm_HandSolder, F.Cu at (268.7, 100.5)
- added R18: 10K, Resistor_SMD:R_0603_1608Metric_Pad0.98x0.95mm_HandSolder, F.Cu at (264.0, 106.1)
- added R19: 200, Resistor_SMD:R_0603_1608Metric_Pad0.98x0.95mm_HandSolder, F.Cu at (278.7, 100.5)
- added R20: 10K, Resistor_SMD:R_0603_1608Metric_Pad0.98x0.95mm_HandSolder, F.Cu at (274.0, 106.1)
- added R21: 200, Resistor_SMD:R_0603_1608Metric_Pad0.98x0.95mm_HandSolder, F.Cu at (288.7, 100.5)
- added R22: 10K, Resistor_SMD:R_0603_1608Metric_Pad0.98x0.95mm_HandSolder, F.Cu at (284.0, 106.1)
- added R23: 200, Resistor_SMD:R_0603_1608Metric_Pad0.98x0.95mm_HandSolder, F.Cu at (298.7, 100.5)
- added R24: 10K, Resistor_SMD:R_0603_1608Metric_Pad0.98x0.95mm_HandSolder, F.Cu at (294.0, 106.1)
- added R5: 200, Resistor_SMD:R_0603_1608Metric_Pad0.98x0.95mm_HandSolder, F.Cu at (138.7, 100.5)
- added R6: 10K, Resistor_SMD:R_0603_1608Metric_Pad0.98x0.95mm_HandSolder, F.Cu at (134.0, 106.1)
- added R7: 200, Resistor_SMD:R_0603_1608Metric_Pad0.98x0.95mm_HandSolder, F.Cu at (148.7, 100.5)
- added R8: 10K, Resistor_SMD:R_0603_1608Metric_Pad0.98x0.95mm_HandSolder, F.Cu at (144.0, 106.1)
- added R9: 200, Resistor_SMD:R_0603_1608Metric_Pad0.98x0.95mm_HandSolder, F.Cu at (158.7, 100.5)
- moved SW1 0.40 mm to (304.2, 96.5)
- moved SW2 0.40 mm to (317.2, 96.5)
Connections:
- U1 pad 10: unconnected-(U1-GPIO7-Pad10) -> /F6
- U1 pad 11: unconnected-(U1-GPIO8-Pad11) -> /F7
- U1 pad 12: unconnected-(U1-GPIO9-Pad12) -> /F8
- U1 pad 14: unconnected-(U1-GPIO10-Pad14) -> /F9
- U1 pad 15: unconnected-(U1-GPIO11-Pad15) -> /F10
- U1 pad 2: unconnected-(U1-GPIO1-Pad2) -> Net-(D35-In)
- U1 pad 36: unconnected-(U1-3V3-Pad36) -> +3.3V
- U1 pad 4: unconnected-(U1-GPIO2-Pad4) -> /F1
- U1 pad 5: unconnected-(U1-GPIO3-Pad5) -> /F2
- U1 pad 6: unconnected-(U1-GPIO4-Pad6) -> /F3
- U1 pad 7: unconnected-(U1-GPIO5-Pad7) -> /F4
- U1 pad 9: unconnected-(U1-GPIO6-Pad9) -> /F5
- U2 pad 25: /F1 -> unconnected-(U2-S7-Pad25)
- U2 pad 26: /F2 -> unconnected-(U2-S8-Pad26)
- U2 pad 4: /F3 -> unconnected-(U2-S16-Pad4)
- U2 pad 5: /F4 -> unconnected-(U2-S15-Pad5)
Routing:
- net +5V: track 906.7 -> 1246.1 mm, vias 1 -> 7
- net +3.3V: track 0.00 -> 283.1 mm, vias 0 -> 1
- net Vref: track 658.4 -> 386.0 mm, vias 4 -> 3
- net Net-(D35-In): track 0.00 -> 117.4 mm, vias 0 -> 1
- net /F10: track 0.00 -> 116.8 mm, vias 0 -> 1
- net /F9: track 0.00 -> 112.1 mm, vias 0 -> 1
- net Net-(D36-Out): track 0.00 -> 105.2 mm, vias 0 -> 2
- net /F8: track 0.00 -> 101.0 mm, vias 0 -> 1
- net /F7: track 0.00 -> 92.6 mm, vias 0 -> 1
- net /F6: track 0.00 -> 86.4 mm, vias 0 -> 1
- net /F5: track 0.00 -> 82.5 mm, vias 0 -> 1
- net Net-(D35-Out): track 0.00 -> 66.0 mm, vias 0 -> 2
- net Net-(D37-Out): track 0.00 -> 66.0 mm, vias 0 -> 2
- net /F4: track 132.7 -> 82.5 mm, vias 0 -> 1
- net /F2: track 139.6 -> 97.7 mm, vias 0 -> 1
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Other:
- board size 268.8 x 136.9 mm -> 270 x 140.9 mm
- board text added: "v1.11"
- board text removed: "v1.0"

Commit message: PCB v1.2 (correct values and signature)
Parts:
- R10, R12, R14, R16, R18, R20, R22, R24, R6, R8: value 10K -> 33K
Other:
- board text added: "Chord Pico v1.2"
- board text added: "github.com/whowechina"
- board text removed: "Chord Pico"
- board text removed: "v1.11"

Commit message: PCB optimization, VBUS for LDO
Connections:
- C17 pad 1: +5V -> VLED
- C18 pad 1: +5V -> VLED
- C19 pad 1: +5V -> VLED
- C20 pad 1: +5V -> VLED
- C21 pad 1: +5V -> VLED
- C22 pad 1: +5V -> VLED
- C23 pad 1: +5V -> VLED
- C24 pad 1: +5V -> VLED
- C25 pad 1: +5V -> VLED
- C26 pad 1: +5V -> VLED
- C27 pad 1: +5V -> VLED
- C28 pad 1: +5V -> VLED
- C29 pad 1: +5V -> VLED
- C30 pad 1: +5V -> VLED
- C31 pad 1: +5V -> VLED
- C32 pad 1: +5V -> VLED
- CC1 pad 1: +5V -> VBUS
- D1 pad V: +5V -> VLED
- D10 pad V: +5V -> VLED
- D11 pad V: +5V -> VLED
- D12 pad V: +5V -> VLED
- D13 pad V: +5V -> VLED
- D14 pad V: +5V -> VLED
- D15 pad V: +5V -> VLED
- D16 pad V: +5V -> VLED
- D17 pad V: +5V -> VLED
- D18 pad V: +5V -> VLED
- D19 pad V: +5V -> VLED
- D2 pad V: +5V -> VLED
- D20 pad V: +5V -> VLED
- D21 pad V: +5V -> VLED
- D22 pad V: +5V -> VLED
- D23 pad V: +5V -> VLED
- D24 pad V: +5V -> VLED
- D25 pad V: +5V -> VLED
- D26 pad V: +5V -> VLED
- D27 pad V: +5V -> VLED
- D28 pad V: +5V -> VLED
- D29 pad V: +5V -> VLED
- D3 pad V: +5V -> VLED
- D30 pad V: +5V -> VLED
- D31 pad V: +5V -> VLED
- D32 pad V: +5V -> VLED
- D33 pad V: +5V -> VLED
- D34 pad V: +5V -> VLED
- D35 pad V: +5V -> VLED
- D36 pad V: +5V -> VLED
- D37 pad V: +5V -> VLED
- D38 pad V: +5V -> VLED
- D39 pad V: +5V -> VLED
- D4 pad V: +5V -> VLED
- D40 pad V: +5V -> VLED
- D41 pad V: +5V -> VLED
- D42 pad V: +5V -> VLED
- D5 pad V: +5V -> VLED
- D6 pad V: +5V -> VLED
- D7 pad V: +5V -> VLED
- D8 pad V: +5V -> VLED
- D9 pad V: +5V -> VLED
- U1 pad 39: +5V -> VLED
- U1 pad 40: Net-(U1-VBUS) -> VBUS
- U7 pad 1: +5V -> VBUS
- U7 pad 3: +5V -> VBUS
- USB1 pad 11: Net-(U1-VBUS) -> VBUS
- USB1 pad 2: Net-(U1-VBUS) -> VBUS
Routing:
- net +5V: track 1246.1 -> 0.00 mm, vias 7 -> 0
- net VLED: track 0.00 -> 1231.1 mm, vias 0 -> 7
- net VBUS: track 0.00 -> 121.2 mm, vias 0 -> 5
- net Net-(U1-VBUS): track 104.9 -> 0.00 mm, vias 3 -> 0
- net Vref: track 386.0 -> 385.3 mm
- net GND: track 25.7 -> 26.1 mm, vias 209 -> 210
Other:
- board text added: "Chord Pico v1.21"
- board text removed: "Chord Pico v1.2"
