File: PCB/plus/chord_plus.kicad_pcb (KiCad board)
At the start: 2 copper layers, 376.3 x 194.5 mm, 127 parts, among them SW1 SW_DIP_x01, SW2 SW_DIP_x01, U1 PiPico, U2 ADG706BRUZ, U6 LM4040DBZ-3, U7 TPS7A2042

Commit message: PCB optimization, VBUS for LDO
Connections:
- C17 pad 1: +5V -> VLED
- C18 pad 1: +5V -> VLED
- C19 pad 1: +5V -> VLED
- C20 pad 1: +5V -> VLED
- C21 pad 1: +5V -> VLED
- C22 pad 1: +5V -> VLED
- C23 pad 1: +5V -> VLED
- C24 pad 1: +5V -> VLED
- C25 pad 1: +5V -> VLED
- C26 pad 1: +5V -> VLED
- C27 pad 1: +5V -> VLED
- C28 pad 1: +5V -> VLED
- C29 pad 1: +5V -> VLED
- C30 pad 1: +5V -> VLED
- C31 pad 1: +5V -> VLED
- C32 pad 1: +5V -> VLED
- CC1 pad 1: +5V -> VBUS
- D1 pad V: +5V -> VLED
- D10 pad V: +5V -> VLED
- D11 pad V: +5V -> VLED
- D12 pad V: +5V -> VLED
- D13 pad V: +5V -> VLED
- D14 pad V: +5V -> VLED
- D15 pad V: +5V -> VLED
- D16 pad V: +5V -> VLED
- D17 pad V: +5V -> VLED
- D18 pad V: +5V -> VLED
- D19 pad V: +5V -> VLED
- D2 pad V: +5V -> VLED
- D20 pad V: +5V -> VLED
- D21 pad V: +5V -> VLED
- D22 pad V: +5V -> VLED
- D23 pad V: +5V -> VLED
- D24 pad V: +5V -> VLED
- D25 pad V: +5V -> VLED
- D26 pad V: +5V -> VLED
- D27 pad V: +5V -> VLED
- D28 pad V: +5V -> VLED
- D29 pad V: +5V -> VLED
- D3 pad V: +5V -> VLED
- D30 pad V: +5V -> VLED
- D31 pad V: +5V -> VLED
- D32 pad V: +5V -> VLED
- D33 pad V: +5V -> VLED
- D34 pad V: +5V -> VLED
- D35 pad V: +5V -> VLED
- D36 pad V: +5V -> VLED
- D37 pad V: +5V -> VLED
- D38 pad V: +5V -> VLED
- D39 pad V: +5V -> VLED
- D4 pad V: +5V -> VLED
- D40 pad V: +5V -> VLED
- D41 pad V: +5V -> VLED
- D42 pad V: +5V -> VLED
- D5 pad V: +5V -> VLED
- D6 pad V: +5V -> VLED
- D7 pad V: +5V -> VLED
- D8 pad V: +5V -> VLED
- D9 pad V: +5V -> VLED
- U1 pad 39: +5V -> VLED
- U1 pad 40: Net-(U1-VBUS) -> VBUS
- U7 pad 1: +5V -> VBUS
- U7 pad 3: +5V -> VBUS
- USB1 pad 11: Net-(U1-VBUS) -> VBUS
- USB1 pad 2: Net-(U1-VBUS) -> VBUS
Routing:
- net +5V: track 1659.0 -> 0.00 mm, vias 5 -> 0
- net VLED: track 0.00 -> 1644.9 mm, vias 0 -> 5
- net VBUS: track 0.00 -> 169.9 mm, vias 0 -> 3
- net Net-(U1-VBUS): track 133.6 -> 0.00 mm, vias 3 -> 0
- net +3.3V: track 369.2 -> 369.7 mm
- net GND: track 18.8 -> 18.4 mm, vias 120 -> 124
Other:
- board text added: "Chord Pico+ v1.01"
- board text removed: "Chord Pico+ v1.0"
