File: PCB/plus/chord_plus.kicad_sch (KiCad schematic)
At the start: 127 parts, among them SW1 SW_DIP_x01, SW2 SW_DIP_x01, U1 PiPico, U2 ADG706BRUZ, U6 LM4040DBZ-3, U7 TPS7A2042

Commit message: PCB optimization, VBUS for LDO
Connections:
- net VBUS: now reaches U1.40 (VBUS), USB1.11 (VBUS), USB1.2 (VBUS)
- net VBUS: now also CC1.1, U7.1 (IN), U7.3 (EN)
- net +5V renamed VLED
- net VLED: no longer CC1.1, U7.1 (IN), U7.3 (EN)
Changed lines of the file:
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@@
 	(paper "A3")
 	(junction
+		(at 158.115 40.64)
+		(diameter 0)
+		(color 0 0 0 0)
+	)
+	(junction
 		(at 372.11 239.395)
 		(diameter 0)
@@
 	)
 	(junction
+		(at 158.115 59.055)
+		(diameter 0)
+		(color 0 0 0 0)
+	)
+	(junction
 		(at 168.91 174.625)
 		(diameter 0)
@@
 	)
 	(junction
-		(at 143.51 59.055)
-		(diameter 0)
-		(color 0 0 0 0)
-	)
-	(junction
 		(at 295.91 208.915)
 		(diameter 0)
@@
 	)
 	(junction
+		(at 134.62 40.64)
+		(diameter 0)
+		(color 0 0 0 0)
+	)
+	(junction
 		(at 69.85 170.18)
 		(diameter 0)
@@
 	)
 	(junction
-		(at 158.115 59.055)
-		(diameter 0)
-		(color 0 0 0 0)
-	)
-	(junction
 		(at 336.55 150.495)
 		(diameter 0)
@@
 	(wire
 		(pts
-			(xy 143.51 59.055) (xy 158.115 59.055)
-		)
-		(stroke
-			(width 0)
-			(type default)
-		)
-	)
-	(wire
-		(pts
 			(xy 237.49 174.625) (xy 245.11 174.625)
 		)
@@
 	(wire
 		(pts
-			(xy 143.51 59.055) (xy 143.51 53.975)
+			(xy 143.51 53.975) (xy 143.51 80.01)
 		)
 		(stroke
@@
 	(wire
 		(pts
+			(xy 158.115 40.64) (xy 158.115 59.055)
+		)
+		(stroke
+			(width 0)
+			(type default)
+		)
+	)
+	(wire
+		(pts
 			(xy 48.26 80.01) (xy 48.26 162.56)
 		)
@@
 	(wire
 		(pts
-			(xy 143.51 80.01) (xy 143.51 59.055)
-		)
-		(stroke
-			(width 0)
-			(type default)
-		)
-	)
-	(wire
-		(pts
 			(xy 285.75 60.325) (xy 285.75 59.055)
 		)
@@
 	(wire
 		(pts
+			(xy 134.62 40.64) (xy 158.115 40.64)
+		)
+		(stroke
+			(width 0)
+			(type default)
+		)
+	)
+	(wire
+		(pts
 			(xy 207.01 102.87) (xy 212.725 102.87)
 		)
@@
 			)
 		)
-		(property "Value" "+5V"
+		(property "Value" "VLED"
 			(at 248.285 220.98 0)
 			(effects
@@
 			)
 		)
-		(property "Value" "+5V"
+		(property "Value" "VLED"
 			(at 143.51 50.165 0)
 			(effects
@@
 			)
 		)
-		(property "Value" "+5V"
+		(property "Value" "VLED"
 			(at 38.735 151.765 0)
 			(effects
@@
 			)
 		)
-		(property "Value" "+5V"
+		(property "Value" "VLED"
 			(at 23.495 193.04 0)
 			(effects
@@
 					(unit 1)
 				)
+			)
+		)
+	)
+	(symbol
+		(lib_id "power:+5V")
+		(at 158.115 40.64 0)
+		(unit 1)
+		(exclude_from_sim no)
+		(in_bom yes)
+		(on_board yes)
+		(dnp no)
+		(property "Reference" "#PWR04"
+			(at 158.115 44.45 0)
+			(effects
+				(font
+					(size 1.27 1.27)
+				)
+				(hide yes)
+			)
+		)
+		(property "Value" "VBUS"
+			(at 158.115 36.83 0)
+			(effects
+				(font
+					(size 1.27 1.27)
+				)
+			)
+		)
+		(property "Footprint" ""
+			(at 158.115 40.64 0)
+			(effects
+				(font
+					(size 1.27 1.27)
+				)
+				(hide yes)
+			)
+		)
+		(property "Datasheet" ""
+			(at 158.115 40.64 0)
+			(effects
+				(font
+					(size 1.27 1.27)
+				)
+				(hide yes)
+			)
+		)
+		(property "Description" "Power symbol creates a global label with name \"+5V\""
+			(at 158.115 40.64 0)
+			(effects
+				(font
+					(size 1.27 1.27)
+				)
+				(hide yes)
+			)
+		)
+		(pin "1"
+		)
+		(instances
+			(project "chord_plus"
+				(path "/2e3f5573-c264-4a8b-a2f0-0e6473d39aad"
+					(reference "#PWR04")
+					(unit 1)
+				)
